File: pcb/kicad/00Key.kicad_pcb (KiCad board)
At the start: 2 copper layers, 304.8 x 170.8 mm, 268 parts, among them Q1 IRLZ44N, U1 Teensy4.1

Commit message: Modified schematic and pcb to use kailh hotswaps rather than MX+LED footprints
Parts:
- removed R_0_1, R_1_1, R_2_1, R_3_1, R_4_1, R_5_1, R_6_1, R_7_1, R_8_1, R_9_1, R_A_1, R_BSLSH_1, R_BSPACE_1, R_B_1, R_CAPS_1, R_COMMA_1, R_C_1, R_DEL_1, R_DOT_1, R_DOWN_1, R_D_1, R_END_1, R_ENTER_1, R_EQUALS_1, R_ESC_1, R_E_1, R_F10_1, R_F11_1, R_F12_1, R_F1_1, R_F2_1, R_F3_1, R_F4_1, R_F5_1, R_F6_1, R_F7_1, R_F8_1, R_F9_1, R_FN_1, R_F_1, R_G_1, R_HOME_1, R_H_1, R_I_1, R_J_1, R_K_1, R_LALT_1, R_LBRAC_1, R_LCTRL_1, R_LEFT_1, R_LSHIFT_1, R_L_1, R_MINUS_1, R_M_1, R_N_1, R_OS_1, R_O_1, R_PAUSE_1, R_PGDN_1, R_PGUP_1, R_PRTSC_1, R_P_1, R_QUOTE_1, R_Q_1, R_RALT_1, R_RBRAC_1, R_RCTRL_1, R_RIGHT_1, R_RSHIFT_1, R_R_1, R_SEMIC_1, R_SLASH_1, R_SPACE_1, R_S_1, R_TAB_1, R_TILDE_1, R_T_1, R_UP_1, R_U_1, R_V_1, R_W_1, R_X_1, R_Y_1, R_Z_1: 470, Resistor_THT:R_Axial_DIN0207_L6.3mm_D2.5mm_P7.62mm_Horizontal
- D_ESC_1: moved to B.Cu
- MX_0_1, MX_1_1, MX_2_1, MX_3_1, MX_4_1, MX_5_1, MX_6_1, MX_7_1, MX_8_1, MX_9_1, MX_A_1, MX_B_1, MX_COMMA_1, MX_C_1, MX_DEL_1, MX_DOT_1, MX_DOWN_1, MX_D_1, MX_END_1, MX_EQUALS_1, MX_ESC_1, MX_E_1, MX_F10_1, MX_F11_1, MX_F12_1, MX_F1_1, MX_F2_1, MX_F3_1, MX_F4_1, MX_F5_1, MX_F6_1, MX_F7_1, MX_F8_1, MX_F9_1, MX_FN_1, MX_F_1, MX_G_1, MX_HOME_1, MX_H_1, MX_I_1, MX_J_1, MX_K_1, MX_LBRAC_1, MX_LEFT_1, MX_L_1, MX_MINUS_1, MX_M_1, MX_N_1, MX_O_1, MX_PAUSE_1, MX_PGDN_1, MX_PGUP_1, MX_PRTSC_1, MX_P_1, MX_QUOTE_1, MX_Q_1, MX_RALT_1, MX_RBRAC_1, MX_RCTRL_1, MX_RIGHT_1, MX_R_1, MX_SEMIC_1, MX_SLASH_1, MX_S_1, MX_TILDE_1, MX_T_1, MX_UP_1, MX_U_1, MX_V_1, MX_W_1, MX_X_1, MX_Y_1, MX_Z_1: value MX-LED -> SW_Hotswap_Kailh_MX; footprint keys:MX-1U -> MX:SW_Hotswap_Kailh_MX_1.00u
- MX_BSLSH_1, MX_TAB_1: value MX-LED -> SW_Hotswap_Kailh_MX; footprint keys:MX-1.5U -> MX:SW_Hotswap_Kailh_MX_1.00u
- MX_BSPACE_1: value MX-LED -> SW_Hotswap_Kailh_MX; footprint keys:MX-2U-ReversedStabilizers -> MX:SW_Hotswap_Kailh_MX_1.00u
- MX_CAPS_1, MX_RSHIFT_1: value MX-LED -> SW_Hotswap_Kailh_MX; footprint keys:MX-1.75U -> MX:SW_Hotswap_Kailh_MX_1.00u
- MX_ENTER_1, MX_LSHIFT_1: value MX-LED -> SW_Hotswap_Kailh_MX; footprint keys:MX-2.25U-ReversedStabilizers -> MX:SW_Hotswap_Kailh_MX_1.00u
- MX_LALT_1, MX_LCTRL_1, MX_OS_1: value MX-LED -> SW_Hotswap_Kailh_MX; footprint keys:MX-1.25U -> MX:SW_Hotswap_Kailh_MX_1.00u
- MX_SPACE_1: value MX-LED -> SW_Hotswap_Kailh_MX; footprint keys:MX-6.25U -> MX:SW_Hotswap_Kailh_MX_1.00u
- moved D_ESC_1 43.3 mm to (48.5, 99.7), turned to 180 degrees
Connections:
- U1 pad 1: Net-(U1-Pad1) -> unconnected-(U1-GND-Pad1)
- U1 pad 10: Net-(U1-Pad10) -> unconnected-(U1-8_TX2_IN1-Pad10)
- U1 pad 11: Net-(U1-Pad11) -> unconnected-(U1-9_OUT1C-Pad11)
- U1 pad 12: Net-(U1-Pad12) -> unconnected-(U1-10_CS_MQSR-Pad12)
- U1 pad 13: Net-(U1-Pad13) -> unconnected-(U1-11_MOSI_CTX1-Pad13)
- U1 pad 14: Net-(U1-Pad14) -> unconnected-(U1-12_MISO_MQSL-Pad14)
- U1 pad 15: Net-(U1-Pad15) -> unconnected-(U1-3V3-Pad15)
- U1 pad 18: Net-(U1-Pad18) -> unconnected-(U1-26_A12_MOSI1-Pad18)
- U1 pad 19: Net-(U1-Pad19) -> unconnected-(U1-27_A13_SCK1-Pad19)
- U1 pad 21: Net-(U1-Pad21) -> unconnected-(U1-29_TX7-Pad21)
- U1 pad 22: Net-(U1-Pad22) -> unconnected-(U1-30_CRX3-Pad22)
- U1 pad 23: Net-(U1-Pad23) -> unconnected-(U1-31_CTX3-Pad23)
- U1 pad 24: Net-(U1-Pad24) -> unconnected-(U1-32_OUT1B-Pad24)
- U1 pad 25: Net-(U1-Pad25) -> unconnected-(U1-33_MCLK2-Pad25)
- U1 pad 26: Net-(U1-Pad26) -> unconnected-(U1-34_RX8-Pad26)
- U1 pad 27: Net-(U1-Pad27) -> unconnected-(U1-35_TX8-Pad27)
- U1 pad 34: Net-(U1-Pad34) -> unconnected-(U1-GND-Pad34)
- U1 pad 35: Net-(U1-Pad35) -> unconnected-(U1-13_SCK_LED-Pad35)
- U1 pad 49: Net-(U1-Pad49) -> unconnected-(U1-VUSB-Pad49)
- U1 pad 50: Net-(U1-Pad50) -> unconnected-(U1-VBAT-Pad50)
- U1 pad 51: Net-(U1-Pad51) -> unconnected-(U1-3V3-Pad51)
- U1 pad 52: Net-(U1-Pad52) -> unconnected-(U1-GND-Pad52)
- U1 pad 53: Net-(U1-Pad53) -> unconnected-(U1-PROGRAM-Pad53)
- U1 pad 54: Net-(U1-Pad54) -> unconnected-(U1-ON_OFF-Pad54)
- U1 pad 55: Net-(U1-Pad55) -> unconnected-(U1-5V-Pad55)
- U1 pad 56: Net-(U1-Pad56) -> unconnected-(U1-D--Pad56)
- U1 pad 57: Net-(U1-Pad57) -> unconnected-(U1-D+-Pad57)
- U1 pad 58: Net-(U1-Pad58) -> unconnected-(U1-GND-Pad58)
- U1 pad 59: Net-(U1-Pad59) -> unconnected-(U1-GND-Pad59)
- U1 pad 60: Net-(U1-Pad60) -> unconnected-(U1-R+-Pad60)
- U1 pad 61: Net-(U1-Pad61) -> unconnected-(U1-LED-Pad61)
- U1 pad 62: Net-(U1-Pad62) -> unconnected-(U1-T--Pad62)
- U1 pad 63: Net-(U1-Pad63) -> unconnected-(U1-T+-Pad63)
- U1 pad 64: Net-(U1-Pad64) -> unconnected-(U1-GND-Pad64)
- U1 pad 65: Net-(U1-Pad65) -> unconnected-(U1-R--Pad65)
- U1 pad 66: Net-(U1-Pad66) -> unconnected-(U1-D--Pad66)
- U1 pad 67: Net-(U1-Pad67) -> unconnected-(U1-D+-Pad67)
- U1 pad 8: Net-(U1-Pad8) -> unconnected-(U1-6_OUT1D-Pad8)
- U1 pad 9: Net-(U1-Pad9) -> unconnected-(U1-7_RX2_OUT1A-Pad9)
Routing:
- net LEDGND: track 1690.6 -> 0.00 mm
- net col0: track 392.2 -> 0.00 mm
- net 5V: track 384.0 -> 0.00 mm
- net col1: track 383.8 -> 0.00 mm
- net col3: track 336.7 -> 0.00 mm
- net col2: track 335.8 -> 0.00 mm
- net row0: track 333.5 -> 0.00 mm
- net row1: track 313.9 -> 0.00 mm
- net row2: track 306.5 -> 0.00 mm
- net GND: track 300.1 -> 0.00 mm
- net row3: track 299.1 -> 0.00 mm
- net col4: track 287.1 -> 0.00 mm
- net row4: track 285.2 -> 0.00 mm
- net row5: track 279.1 -> 0.00 mm
- net col5: track 273.5 -> 0.00 mm, vias 1 -> 0
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
Commit message: Change diodes to smd, moved them to under switches, replaced teensy with header pins, reduced size of pcb
Parts:
- removed OLED1: SSD1306, oled:128x64OLED
- removed Q1: IRLZ44N, Package_TO_SOT_THT:TO-220-3_Vertical
- removed R_Q1_GATE_1: 10K, Resistor_THT:R_Axial_DIN0207_L6.3mm_D2.5mm_P7.62mm_Horizontal
- removed U1: Teensy4.1, teensy:Teensy41
- added J1: Conn_01x12, Connector_PinSocket_2.54mm:PinSocket_1x12_P2.54mm_Horizontal, B.Cu at (121.1, 206.2)
- added J2: Conn_01x12, Connector_PinSocket_2.54mm:PinSocket_1x12_P2.54mm_Horizontal, B.Cu at (190.9, 206.2)
- D_0_1, D_1_1, D_2_1, D_3_1, D_4_1, D_5_1, D_6_1, D_7_1, D_8_1, D_9_1, D_A_1, D_BSLSH_1, D_BSPACE_1, D_B_1, D_CAPS_1, D_COMMA_1, D_C_1, D_DEL_1, D_DOT_1, D_DOWN_1, D_D_1, D_END_1, D_ENTER_1, D_EQUALS_1, D_E_1, D_F10_1, D_F11_1, D_F12_1, D_F1_1, D_F2_1, D_F3_1, D_F4_1, D_F5_1, D_F6_1, D_F7_1, D_F8_1, D_F9_1, D_FN_1, D_F_1, D_G_1, D_HOME_1, D_H_1, D_I_1, D_J_1, D_K_1, D_LALT_1, D_LBRAC_1, D_LCTRL_1, D_LEFT_1, D_LSHIFT_1, D_L_1, D_MINUS_1, D_M_1, D_N_1, D_OS_1, D_O_1, D_PAUSE_1, D_PGDN_1, D_PGUP_1, D_PRTSC_1, D_P_1, D_QUOTE_1, D_Q_1, D_RALT_1, D_RBRAC_1, D_RCTRL_1, D_RIGHT_1, D_RSHIFT_1, D_R_1, D_SEMIC_1, D_SLASH_1, D_SPACE_1, D_S_1, D_TAB_1, D_TILDE_1, D_T_1, D_UP_1, D_U_1, D_V_1, D_W_1, D_X_1, D_Y_1, D_Z_1: footprint parts:D_SOD123_axial -> Diode_SMD:D_SOD-123; moved to B.Cu
- D_ESC_1: footprint parts:D_SOD123_axial -> Diode_SMD:D_SOD-123
- moved D_RIGHT_1 168.4 mm to (334.9, 196.2), turned to 180 degrees
- moved D_DOWN_1 165.0 mm to (315.8, 196.2), turned to 180 degrees
- moved D_LEFT_1 162.2 mm to (296.8, 196.2), turned to 180 degrees
- moved D_RCTRL_1 159.7 mm to (277.7, 196.2), turned to 180 degrees
- moved D_FN_1 159.1 mm to (258.7, 196.2), turned to 180 degrees
- moved D_RALT_1 157.8 mm to (239.6, 196.2), turned to 180 degrees
- moved D_SPACE_1 153.5 mm to (170.7, 196.2), turned to 180 degrees
- moved D_END_1 151.5 mm to (334.9, 177.2), turned to 180 degrees
- moved D_LALT_1 149.3 mm to (99.3, 196.2), turned to 180 degrees
- moved D_UP_1 147.9 mm to (315.8, 177.2), turned to 180 degrees
- moved D_LCTRL_1 147.4 mm to (51.6, 196.2), turned to 180 degrees
- moved D_OS_1 145.7 mm to (75.4, 196.2), turned to 180 degrees
- moved D_SLASH_1 142.7 mm to (263.5, 177.2), turned to 180 degrees
- moved D_RSHIFT_1 141.4 mm to (289.7, 177.2), turned to 180 degrees
- moved D_DOT_1 141.1 mm to (244.5, 177.2), turned to 180 degrees
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Other:
- board size 304.8 x 170.8 mm -> 304.8 x 114.3 mm
