File: pcb/kicad/switches.kicad_sch (KiCad schematic)
At the start: 252 parts

Commit message: Modified schematic and pcb to use kailh hotswaps rather than MX+LED footprints
Parts:
- removed R_0_1, R_1_1, R_2_1, R_3_1, R_4_1, R_5_1, R_6_1, R_7_1, R_8_1, R_9_1, R_A_1, R_BSLSH_1, R_BSPACE_1, R_B_1, R_CAPS_1, R_COMMA_1, R_C_1, R_DEL_1, R_DOT_1, R_DOWN_1, R_D_1, R_END_1, R_ENTER_1, R_EQUALS_1, R_ESC_1, R_E_1, R_F10_1, R_F11_1, R_F12_1, R_F1_1, R_F2_1, R_F3_1, R_F4_1, R_F5_1, R_F6_1, R_F7_1, R_F8_1, R_F9_1, R_FN_1, R_F_1, R_G_1, R_HOME_1, R_H_1, R_I_1, R_J_1, R_K_1, R_LALT_1, R_LBRAC_1, R_LCTRL_1, R_LEFT_1, R_LSHIFT_1, R_L_1, R_MINUS_1, R_M_1, R_N_1, R_OS_1, R_O_1, R_PAUSE_1, R_PGDN_1, R_PGUP_1, R_PRTSC_1, R_P_1, R_QUOTE_1, R_Q_1, R_RALT_1, R_RBRAC_1, R_RCTRL_1, R_RIGHT_1, R_RSHIFT_1, R_R_1, R_SEMIC_1, R_SLASH_1, R_SPACE_1, R_S_1, R_TAB_1, R_TILDE_1, R_T_1, R_UP_1, R_U_1, R_V_1, R_W_1, R_X_1, R_Y_1, R_Z_1: (no value), symbol Device:R
- D_0_1, D_1_1, D_2_1, D_3_1, D_4_1, D_5_1, D_6_1, D_7_1, D_8_1, D_9_1, D_A_1, D_BSLSH_1, D_BSPACE_1, D_B_1, D_CAPS_1, D_COMMA_1, D_C_1, D_DEL_1, D_DOT_1, D_DOWN_1, D_D_1, D_END_1, D_ENTER_1, D_EQUALS_1, D_ESC_1, D_E_1, D_F10_1, D_F11_1, D_F12_1, D_F1_1, D_F2_1, D_F3_1, D_F4_1, D_F5_1, D_F6_1, D_F7_1, D_F8_1, D_F9_1, D_FN_1, D_F_1, D_G_1, D_HOME_1, D_H_1, D_I_1, D_J_1, D_K_1, D_LALT_1, D_LBRAC_1, D_LCTRL_1, D_LEFT_1, D_LSHIFT_1, D_L_1, D_MINUS_1, D_M_1, D_N_1, D_OS_1, D_O_1, D_PAUSE_1, D_PGDN_1, D_PGUP_1, D_PRTSC_1, D_P_1, D_QUOTE_1, D_Q_1, D_RALT_1, D_RBRAC_1, D_RCTRL_1, D_RIGHT_1, D_RSHIFT_1, D_R_1, D_SEMIC_1, D_SLASH_1, D_SPACE_1, D_S_1, D_TAB_1, D_TILDE_1, D_T_1, D_UP_1, D_U_1, D_V_1, D_W_1, D_X_1, D_Y_1, D_Z_1: value (none) -> D; footprint (none) -> parts:D_SOD123_axial
- MX_0_1, MX_1_1, MX_2_1, MX_3_1, MX_4_1, MX_5_1, MX_6_1, MX_7_1, MX_8_1, MX_9_1, MX_A_1, MX_BSLSH_1, MX_BSPACE_1, MX_B_1, MX_CAPS_1, MX_COMMA_1, MX_C_1, MX_DEL_1, MX_DOT_1, MX_DOWN_1, MX_D_1, MX_END_1, MX_ENTER_1, MX_EQUALS_1, MX_ESC_1, MX_E_1, MX_F10_1, MX_F11_1, MX_F12_1, MX_F1_1, MX_F2_1, MX_F3_1, MX_F4_1, MX_F5_1, MX_F6_1, MX_F7_1, MX_F8_1, MX_F9_1, MX_FN_1, MX_F_1, MX_G_1, MX_HOME_1, MX_H_1, MX_I_1, MX_J_1, MX_K_1, MX_LALT_1, MX_LBRAC_1, MX_LCTRL_1, MX_LEFT_1, MX_LSHIFT_1, MX_L_1, MX_MINUS_1, MX_M_1, MX_N_1, MX_OS_1, MX_O_1, MX_PAUSE_1, MX_PGDN_1, MX_PGUP_1, MX_PRTSC_1, MX_P_1, MX_QUOTE_1, MX_Q_1, MX_RALT_1, MX_RBRAC_1, MX_RCTRL_1, MX_RIGHT_1, MX_RSHIFT_1, MX_R_1, MX_SEMIC_1, MX_SLASH_1, MX_SPACE_1, MX_S_1, MX_TAB_1, MX_TILDE_1, MX_T_1, MX_UP_1, MX_U_1, MX_V_1, MX_W_1, MX_X_1, MX_Y_1, MX_Z_1: value (none) -> SW_Hotswap_Kailh_MX; footprint (none) -> MX:SW_Hotswap_Kailh_MX_1.00u; symbol 00Key-rescue:MX-LED-keys -> MX_keys:SW_Hotswap_Kailh_MX
Connections:
- net LEDGND: no longer MX_0_1.4 (LEDGND), MX_1_1.4 (LEDGND), MX_2_1.4 (LEDGND), MX_3_1.4 (LEDGND), MX_4_1.4 (LEDGND), MX_5_1.4 (LEDGND), MX_6_1.4 (LEDGND), MX_7_1.4 (LEDGND), MX_8_1.4 (LEDGND), MX_9_1.4 (LEDGND), MX_A_1.4 (LEDGND), MX_BSLSH_1.4 (LEDGND), MX_BSPACE_1.4 (LEDGND), MX_B_1.4 (LEDGND), MX_CAPS_1.4 (LEDGND), MX_COMMA_1.4 (LEDGND), MX_C_1.4 (LEDGND), MX_DEL_1.4 (LEDGND), MX_DOT_1.4 (LEDGND), MX_DOWN_1.4 (LEDGND), MX_D_1.4 (LEDGND), MX_END_1.4 (LEDGND), MX_ENTER_1.4 (LEDGND), MX_EQUALS_1.4 (LEDGND), MX_ESC_1.4 (LEDGND), MX_E_1.4 (LEDGND), MX_F10_1.4 (LEDGND), MX_F11_1.4 (LEDGND), MX_F12_1.4 (LEDGND), MX_F1_1.4 (LEDGND), MX_F2_1.4 (LEDGND), MX_F3_1.4 (LEDGND), MX_F4_1.4 (LEDGND), MX_F5_1.4 (LEDGND), MX_F6_1.4 (LEDGND), MX_F7_1.4 (LEDGND), MX_F8_1.4 (LEDGND), MX_F9_1.4 (LEDGND), MX_FN_1.4 (LEDGND), MX_F_1.4 (LEDGND), MX_G_1.4 (LEDGND), MX_HOME_1.4 (LEDGND), MX_H_1.4 (LEDGND), MX_I_1.4 (LEDGND), MX_J_1.4 (LEDGND), MX_K_1.4 (LEDGND), MX_LALT_1.4 (LEDGND), MX_LBRAC_1.4 (LEDGND), MX_LCTRL_1.4 (LEDGND), MX_LEFT_1.4 (LEDGND), MX_LSHIFT_1.4 (LEDGND), MX_L_1.4 (LEDGND), MX_MINUS_1.4 (LEDGND), MX_M_1.4 (LEDGND), MX_N_1.4 (LEDGND), MX_OS_1.4 (LEDGND), MX_O_1.4 (LEDGND), MX_PAUSE_1.4 (LEDGND), MX_PGDN_1.4 (LEDGND), MX_PGUP_1.4 (LEDGND), MX_PRTSC_1.4 (LEDGND), MX_P_1.4 (LEDGND), MX_QUOTE_1.4 (LEDGND), MX_Q_1.4 (LEDGND), MX_RALT_1.4 (LEDGND), MX_RBRAC_1.4 (LEDGND), MX_RCTRL_1.4 (LEDGND), MX_RIGHT_1.4 (LEDGND), MX_RSHIFT_1.4 (LEDGND), MX_R_1.4 (LEDGND), MX_SEMIC_1.4 (LEDGND), MX_SLASH_1.4 (LEDGND), MX_SPACE_1.4 (LEDGND), MX_S_1.4 (LEDGND), MX_TAB_1.4 (LEDGND), MX_TILDE_1.4 (LEDGND), MX_T_1.4 (LEDGND), MX_UP_1.4 (LEDGND), MX_U_1.4 (LEDGND), MX_V_1.4 (LEDGND), MX_W_1.4 (LEDGND), MX_X_1.4 (LEDGND), MX_Y_1.4 (LEDGND), MX_Z_1.4 (LEDGND)

Commit message: Change diodes to smd, moved them to under switches, replaced teensy with header pins, reduced size of pcb
Parts:
- D_0_1, D_1_1, D_2_1, D_3_1, D_4_1, D_5_1, D_6_1, D_7_1, D_8_1, D_9_1, D_A_1, D_BSLSH_1, D_BSPACE_1, D_B_1, D_CAPS_1, D_COMMA_1, D_C_1, D_DEL_1, D_DOT_1, D_DOWN_1, D_D_1, D_END_1, D_ENTER_1, D_EQUALS_1, D_ESC_1, D_E_1, D_F10_1, D_F11_1, D_F12_1, D_F1_1, D_F2_1, D_F3_1, D_F4_1, D_F5_1, D_F6_1, D_F7_1, D_F8_1, D_F9_1, D_FN_1, D_F_1, D_G_1, D_HOME_1, D_H_1, D_I_1, D_J_1, D_K_1, D_LALT_1, D_LBRAC_1, D_LCTRL_1, D_LEFT_1, D_LSHIFT_1, D_L_1, D_MINUS_1, D_M_1, D_N_1, D_OS_1, D_O_1, D_PAUSE_1, D_PGDN_1, D_PGUP_1, D_PRTSC_1, D_P_1, D_QUOTE_1, D_Q_1, D_RALT_1, D_RBRAC_1, D_RCTRL_1, D_RIGHT_1, D_RSHIFT_1, D_R_1, D_SEMIC_1, D_SLASH_1, D_SPACE_1, D_S_1, D_TAB_1, D_TILDE_1, D_T_1, D_UP_1, D_U_1, D_V_1, D_W_1, D_X_1, D_Y_1, D_Z_1: footprint parts:D_SOD123_axial -> Diode_SMD:D_SOD-123; symbol Device:D -> Diode:1N4148W
